Commit message: chore: update urdf

File: pixkit_description/urdf/vehicle.xacro (robot description, xacro)
@@ -6,5 +6,5 @@
   <link name="base_link">
     <visual>
-      <origin xyz="${vehicle_info['/**']['ros__parameters']['wheel_base']*0.0} 0 0.1" rpy="0 0 ${pi/2.0}"/>
+      <origin xyz="-2.0 0.0 0.1" rpy="0 0 ${pi/2.0}"/>
       <geometry>
         <mesh filename="package://pixkit_description/mesh/hooke.dae" scale="0.001 0.001 0.001"/>

Commit message: fix: mpc trajectory is in front of the model in rviz" -m "if we select init pose in rviz and we found the initial pose is separate from the model. and the mpc trajectory is also in front of the model

File: pixkit_description/urdf/vehicle.xacro (robot description, xacro)
@@ -6,5 +6,5 @@
   <link name="base_link">
     <visual>
-      <origin xyz="-2.0 0.0 0.1" rpy="0 0 ${pi/2.0}"/>
+      <origin xyz="-0.25 0.0 0.1" rpy="0 0 ${pi/2.0}"/>
       <geometry>
         <mesh filename="package://pixkit_description/mesh/hooke.dae" scale="0.001 0.001 0.001"/>
